File: kicad/atmega-gpib.sch (KiCad schematic (older format))
At the start: 18 parts, among them IC1 ATMEGA168PA-P, P2 GPIB, P3 USB_B, U1 FT230XS

Commit message: interim schematic update commit
Parts:
- removed U1: FT230XS, Housings_SSOP:SSOP-16_3.9x4.9mm_Pitch0.635mm, symbol FT230XS
- added J?: USB, symbol USB
- added U?: FT230XS, ~, symbol FT230XS
Other:
- moved on the sheet: P2
Changed lines of the file:
@@
 EESchema Schematic File Version 2
+LIBS:PL_connectors
+LIBS:PL_opamps
+LIBS:PL_comms
+LIBS:PL_microcontrollers
 LIBS:PL_power
-LIBS:FT230X
 LIBS:PL_GPIB
-LIBS:PL_analog_ICs
-LIBS:PL_capacitors
-LIBS:PL_connectors
-LIBS:PL_diodes
-LIBS:PL_displays
-LIBS:PL_inductors
-LIBS:PL_LEDs
-LIBS:PL_microcontrollers
-LIBS:PL_mounting_holes
-LIBS:PL_opamps
-LIBS:PL_opto
-LIBS:PL_references
-LIBS:PL_regulators
-LIBS:PL_relays
-LIBS:PL_resistors
-LIBS:PL_switchers
 LIBS:PL_switches
 LIBS:PL_transistors
+LIBS:PL_regulators
+LIBS:PL_diodes
+LIBS:PL_resistors
+LIBS:PL_capacitors
+LIBS:PL_switchers
+LIBS:PL_opto
+LIBS:PL_inductors
+LIBS:PL_references
+LIBS:PL_relays
+LIBS:PL_displays
+LIBS:PL_analog_ICs
+LIBS:PL_mounting_holes
+LIBS:PL_LEDs
 LIBS:power
 LIBS:device
@@
 LIBS:valves
 LIBS:atmega-gpib-cache
-EELAYER 25 0
+EELAYER 27 0
 EELAYER END
 $Descr A4 11693 8268
@@
 Sheet 1 1
 Title ""
-Date ""
+Date "1 jun 2017"
 Rev ""
 Comp ""
@@
 	3550 1650 4600 1650
 Wire Wire Line
-	6000 3350 5900 3350
-Wire Wire Line
-	6000 2650 6000 3450
-Wire Wire Line
-	5900 3250 6000 3250
-Connection ~ 6000 3350
-Wire Wire Line
-	5900 3150 6000 3150
-Connection ~ 6000 3250
-Wire Wire Line
-	5900 3050 6000 3050
-Connection ~ 6000 3150
-Wire Wire Line
-	5900 2950 6000 2950
-Connection ~ 6000 3050
-Wire Wire Line
-	5900 2850 6000 2850
-Connection ~ 6000 2950
-Wire Wire Line
-	5900 2750 6000 2750
-Connection ~ 6000 2850
-Wire Wire Line
-	5900 2650 6000 2650
-Connection ~ 6000 2750
+	5900 3350 5800 3350
+Wire Wire Line
+	5900 2650 5900 3450
+Wire Wire Line
+	5800 3250 5900 3250
+Connection ~ 5900 3350
+Wire Wire Line
+	5800 3150 5900 3150
+Connection ~ 5900 3250
+Wire Wire Line
+	5800 3050 5900 3050
+Connection ~ 5900 3150
+Wire Wire Line
+	5800 2950 5900 2950
+Connection ~ 5900 3050
+Wire Wire Line
+	5800 2850 5900 2850
+Connection ~ 5900 2950
+Wire Wire Line
+	5800 2750 5900 2750
+Connection ~ 5900 2850
+Wire Wire Line
+	5800 2650 5900 2650
+Connection ~ 5900 2750
 Text GLabel 3650 3350 2    40   Input ~ 0
 TX
@@
 	1550 3850 1650 3850
 Connection ~ 1550 3950
-NoConn ~ 1650 2050
+NoConn ~ 1650 2250
 $Comp
 L USB_B P3
@@
 	0    -1   1    0
 $EndComp
-$Comp
-L FT230XS U1
-U 1 1 59101FDC
-P 8900 5350
-F 0 "U1" H 8450 5900 50  0000 L CNN
-F 1 "FT230XS" H 9350 5900 50  0000 R CNN
-F 2 "Housings_SSOP:SSOP-16_3.9x4.9mm_Pitch0.635mm" H 8900 5350 50  0001 C CNN
-F 3 "DOCUMENTATION" H 8900 5350 50  0001 C CNN
-	1    8900 5350
-	1    0    0    -1
-$EndComp
-Text GLabel 9650 4950 2    40   Input ~ 0
+Text GLabel 9550 4950 2    40   Input ~ 0
 TX
-Text GLabel 9650 5050 2    40   Input ~ 0
+Text GLabel 9550 5050 2    40   Input ~ 0
 RX
 Wire Wire Line
-	9550 4950 9650 4950
-Wire Wire Line
-	9550 5050 9650 5050
+	9450 4950 9550 4950
+Wire Wire Line
+	9450 5050 9550 5050
 Text GLabel 7350 4750 1    40   Input ~ 0
 5V
@@
 	8150 5750 8250 5750
 Connection ~ 8150 5850
-Wire Wire Line
-	8250 5050 8250 5250
 $Comp
 L C_CER C7
@@
 Wire Wire Line
 	1300 1650 1300 1550
-Connection ~ 8250 5150
 $Comp
 L GPIB P2
 U 1 1 59104927
-P 5250 2450
-F 0 "P2" H 4800 3400 40  0000 L CNN
-F 1 "GPIB" H 5700 3400 40  0000 R CNN
-F 2 "gpib_conn_male:gpib_conn_male" H 4850 2550 60  0001 C CNN
-F 3 "" H 4850 2550 60  0000 C CNN
-	1    5250 2450
+P 5200 2450
+F 0 "P2" H 4750 3400 40  0000 L CNN
+F 1 "GPIB" H 5650 3400 40  0000 R CNN
+F 2 "gpib_conn_male:gpib_conn_male" H 4800 2550 60  0001 C CNN
+F 3 "" H 4800 2550 60  0000 C CNN
+	1    5200 2450
 	1    0    0    -1
 $EndComp
@@
 Wire Wire Line
 	6650 5650 6650 5750
-NoConn ~ 9550 5850
-NoConn ~ 9550 5550
+NoConn ~ 9450 5850
+NoConn ~ 9450 5550
 $Comp
 L FERRITE_BEAD FB1
@@
 L GND #PWR01
 U 1 1 591088AE
-P 6000 3450
-F 0 "#PWR01" H 6000 3250 50  0001 C CNN
-F 1 "GND" H 6000 3350 40  0000 C CNN
-F 2 "" H 6000 3450 50  0000 C CNN
-F 3 "" H 6000 3450 50  0000 C CNN
-	1    6000 3450
+P 5900 3450
+F 0 "#PWR01" H 5900 3250 50  0001 C CNN
+F 1 "GND" H 5900 3350 40  0000 C CNN
+F 2 "" H 5900 3450 50  0000 C CNN
+F 3 "" H 5900 3450 50  0000 C CNN
+	1    5900 3450
 	1    0    0    -1
 $EndComp
@@
 	10150 5550 10150 5650
 Wire Wire Line
-	10150 5650 9550 5650
+	10150 5650 9450 5650
 $Comp
 L LED D2
@@
 	10450 5550 10450 5750
 Wire Wire Line
-	10450 5750 9550 5750
+	10450 5750 9450 5750
 Text GLabel 7950 5050 0    40   Input ~ 0
 VCCIO
@@
 Wire Wire Line
 	3550 3550 3650 3550
-Text GLabel 9650 5250 2    40   Input ~ 0
+Text GLabel 9550 5250 2    40   Input ~ 0
 RTS
-Text GLabel 9650 5350 2    40   Input ~ 0
+Text GLabel 9550 5350 2    40   Input ~ 0
 CTS
 Wire Wire Line
-	9550 5250 9650 5250
-Wire Wire Line
-	9550 5350 9650 5350
+	9450 5250 9550 5250
+Wire Wire Line
+	9450 5350 9550 5350
 Text GLabel 6650 5350 2    40   Input ~ 0
 5V_EXT
@@
 	1300 1650 1650 1650
 Wire Wire Line
-	1650 1850 1600 1850
-Wire Wire Line
-	1600 1850 1600 1650
+	1600 1650 1600 1950
 Connection ~ 1600 1650
 Wire Wire Line
@@
 NoConn ~ 3550 2250
 NoConn ~ 3550 3650
+$Comp
+L FT230XS U?
+U 1 1 592F9057
+P 8850 5350
+F 0 "U?" H 8400 5900 40  0000 L CNN
+F 1 "FT230XS" H 9300 5900 40  0000 R CNN
+F 2 "~" H 8850 5350 60  0000 C CNN
+F 3 "~" H 8850 5350 60  0000 C CNN
+	1    8850 5350
+	1    0    0    -1
+$EndComp
+Wire Wire Line
+	8250 5050 8250 5250
+Connection ~ 8250 5150
+Wire Wire Line
+	1600 1950 1650 1950
+$Comp
+L USB J?
+U 1 1 592F93C4
+P 5400 5650
+F 0 "J?" H 5350 6050 60  0000 C CNN
+F 1 "USB" V 5150 5800 60  0000 C CNN
+F 2 "" H 5400 5650 60  0000 C CNN
+F 3 "" H 5400 5650 60  0000 C CNN
+	1    5400 5650
+	1    0    0    -1
+$EndComp
 $EndSCHEMATC

Commit message: Working on board v2
Parts:
- removed J?: USB, symbol USB
- removed P3: USB_B, w_conn_pc:conn_usb_B, symbol USB_B
- removed U?: FT230XS, ~, symbol FT230XS
- added C4, C9: 0.1uF, PL_capacitors:CERCAP_2_059B_0805, symbol C_CER
- added D3: ERR LED, PL_LEDs:LED_3MM_069A, symbol LED
- added J1: USB_B, symbol USB_B
- added P1: CONN_4X1, ~, symbol CONN_4X1
- added P3: CONN_2X1, ~, symbol CONN_2X1
- added R5: 330, PL_resistors:R_AXIAL_0W25_059A_PL, symbol R_0W25
- added U1: MCP2221A, ~, symbol MCP2221A
- D1: value RX LED -> TX LED
- D2: value TX LED -> RX LED
Connections:
- net labels added: ERR_LED, JMP1
- net labels removed: 5V_EXT, CTS, RTS, VCCIO
- wire segments 125 -> 127
- no-connect marks 5 -> 7
Other:
- note added: "Config jumper"
- note added: "Error LED"
- note added: "Serial TTL Pinout"
- note added: "The datasheet calls for a ceramic cap\nof between 0.22 and 0.47uF on VUSB."
- note removed: "GPIB"
- moved on the sheet: C1, C2, C3, C5, C6, C7, D1, D2, FB1, IC1, P2, R1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

Commit message: v2 board
Parts:
- removed C4: 0.1uF, PL_capacitors:CERCAP_2_059B_0805, symbol C_CER
Connections:
- wire segments 127 -> 126
Other:
- note added: "GPIB-USB adapter"
- moved on the sheet: C2, C3, C5, C6, C7, C8, C9, D1, D2, FB1, J1, R1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
