File: kicad/atmega-gpib.kicad_pcb (KiCad board)
At the start: 2 copper layers, 49.5 x 49.5 mm, 19 parts, among them IC1 ATMEGA328, P2 GPIB, P3 USB_B, U1 FT230XS

Commit message: v2 board
Parts:
- removed the G*** at (137.8, 75.6)
- removed P3: USB_B, w_conn_pc:conn_usb_B
- removed RX: RX LED, PL_LEDs:LED_3MM_069A
- removed TX: TX LED, PL_LEDs:LED_3MM_069A
- added C9: 0.1uF, CERCAP_15_059B_0805, F.Cu at (55.9, 403.9)
- added D1: TX, LED_3MM_069A, F.Cu at (71.1, 405.8)
- added D2: RX, LED_3MM_069A, F.Cu at (66.0, 405.8)
- added D3: ERR, LED_3MM_069A, F.Cu at (83.2, 377.2)
- added G***: OSHW-logo_silkscreen-back_4mm, OSHW-logo_silkscreen-back_4mm, F.Cu at (82.5, 370.8)
- added J1: USB_B, USB_B, F.Cu at (86.4, 400.1)
- added JMP1: CONN_2X1, SIL-2, F.Cu at (68.6, 390.5)
- added P1: CONN_4X1, SIL-4, F.Cu at (49.5, 407.7)
- added R5: 330, R_AXIAL_0W25_059A_PL, F.Cu at (79.4, 386.7)
- C1, C2, C5, C6, C7, C8: footprint PL_capacitors:CERCAP_2_059B_0805 -> CERCAP_15_059B_0805
- C3: footprint PL_capacitors:ELCAP_10_20_V_059A -> ELCAP_10_20_V_059A
- FB1: value FERRITE_BEAD -> FERRITE; footprint PL_inductors:FERRITE_AXIAL_04_069A -> FERRITE_AXIAL_04_069A
- IC1: value ATMEGA328 -> ATMEGA168PA-P
- P2: footprint gpib_conn_male:gpib_conn_male -> 112-024-113R001
- R1, R2, R3, R4: footprint PL_resistors:R_AXIAL_0W25_059A_PL -> R_AXIAL_0W25_059A_PL
- U1: value FT230XS -> MCP2221A; footprint Housings_SSOP:SSOP-16_3.9x4.9mm_Pitch0.635mm -> DIP14_PL
- moved C8 324.4 mm to (58.4, 403.9), turned to 270 degrees
- moved C5 316.4 mm to (77.5, 401.3), turned to 270 degrees
- moved IC1 314.4 mm to (43.2, 387.4)
- moved P2 314.4 mm to (65.4, 370.8)
- moved U1 314.4 mm to (58.4, 392.4), turned to 180 degrees
- moved C1 314.1 mm to (43.9, 389.9)
- moved R3 312.5 mm to (63.5, 402.6), turned to 0 degrees
- moved C7 312.4 mm to (64.8, 390.5), turned to 180 degrees
- moved C6 311.4 mm to (77.5, 398.8), turned to 90 degrees
- moved R1 310.8 mm to (63.5, 397.5)
- moved R4 307.5 mm to (63.5, 400.1), turned to 0 degrees
- moved R2 305.8 mm to (63.5, 395.0)
- moved C3 302.4 mm to (80.0, 389.3), turned to 270 degrees
- moved C2 295.8 mm to (85.1, 390.5), turned to 0 degrees
- moved FB1 289.7 mm to (87.6, 382.3)
Connections:
- net 5V_EXT renamed N-0000041
- C8 pad 1: VCCIO -> N-0000015
- IC1 pad 10: Net-(IC1-Pad10) -> (no net)
- IC1 pad 19: Net-(IC1-Pad19) -> ERR_LED
- IC1 pad 21: Net-(IC1-Pad21) -> (no net)
- IC1 pad 4: CTS -> JMP1
- IC1 pad 5: RTS -> N-0000030
- IC1 pad 6: Net-(IC1-Pad6) -> N-000004
- IC1 pad 9: Net-(IC1-Pad9) -> (no net)
- P2 pad 17: Net-(IC1-Pad19) -> N-0000030
- P2 pad 5: Net-(IC1-Pad10) -> N-000004
- R1 pad 1: Net-(R1-Pad1) -> N-0000019
- R2 pad 1: Net-(R2-Pad1) -> N-0000039
- R3 pad 1: Net-(D1-Pad1) -> N-0000020
- R3 pad 2: VCCIO -> N-0000037
- R4 pad 1: Net-(D2-Pad1) -> N-000009
- R4 pad 2: VCCIO -> N-0000010
- U1 pad 1: TX -> 5V
- U1 pad 10: VCCIO -> (no net)
- U1 pad 11: VCCIO -> N-0000015
- U1 pad 12: 5V -> N-0000039
- U1 pad 13: GND -> N-0000019
- U1 pad 14: Net-(D1-Pad2) -> GND
- U1 pad 2: RTS -> N-0000020
- U1 pad 3: VCCIO -> N-000009
- U1 pad 4: RX -> 5V
- U1 pad 5: GND -> TX
- U1 pad 6: CTS -> RX
- U1 pad 7: Net-(D2-Pad2) -> (no net)
- U1 pad 8: Net-(R2-Pad1) -> (no net)
- U1 pad 9: Net-(R1-Pad1) -> (no net)
Routing:
- net 5V: track 59.5 -> 125.1 mm
- net N-0000041: track 57.0 -> 13.9 mm
- net Net-(D1-Pad2): track 39.1 -> 0.00 mm
- net N-0000030: track 0.00 -> 30.4 mm, vias 0 -> 2
- net VCCIO: track 26.9 -> 0.00 mm, vias 2 -> 0
- net Net-(D2-Pad2): track 25.7 -> 0.00 mm, vias 2 -> 0
- net N-0000020: track 0.00 -> 23.7 mm
- net ERR_LED: track 0.00 -> 23.0 mm, vias 0 -> 2
- net N-000004: track 0.00 -> 23.0 mm, vias 0 -> 2
- net N-000009: track 0.00 -> 22.4 mm
- net JMP1: track 0.00 -> 19.5 mm, vias 0 -> 2
- net CTS: track 18.2 -> 0.00 mm, vias 2 -> 0
- net Net-(IC1-Pad10): track 15.4 -> 0.00 mm
- net N-0000010: track 0.00 -> 15.4 mm
- net N-0000039: track 0.00 -> 13.4 mm
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Other:
- outline, holes or cut-outs redrawn
- board text added: "(v2)"
- board text added: "5V"
- board text added: "GND"
- board text added: "RX"
- board text added: "TX"
- board text removed: "(v1)"

Commit message: Fixing drill file offset
Parts:
- moved R2 296.5 mm to (140.3, 108.6)
- moved C1 296.5 mm to (120.8, 103.5)
- moved C2 296.5 mm to (161.9, 104.1)
- moved C3 296.5 mm to (156.8, 102.9)
- moved C5 296.5 mm to (154.3, 114.9)
- moved C6 296.5 mm to (154.3, 112.4)
- moved C7 296.5 mm to (141.6, 104.1)
- moved C8 296.5 mm to (135.3, 117.5)
- moved C9 296.5 mm to (132.7, 117.5)
- moved D1 296.5 mm to (148.0, 119.4)
- moved D2 296.5 mm to (142.9, 119.4)
- moved D3 296.5 mm to (160.0, 90.8)
- moved FB1 296.5 mm to (164.5, 95.9)
- moved G*** 296.5 mm to (159.4, 84.5)
- moved IC1 296.5 mm to (120.0, 101.0)
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
Commit message: Fixing drill offsets again
Parts:
- moved C7 8.13 mm to (148.0, 109.2)
- moved G*** 8.13 mm to (165.7, 89.5)
- moved P1 8.13 mm to (132.7, 126.4)
- moved C8 8.13 mm to (141.6, 122.6)
- moved C9 8.13 mm to (139.1, 122.6)
- moved R2 8.13 mm to (146.7, 113.7)
- moved C1 8.13 mm to (127.1, 108.6)
- moved C2 8.13 mm to (168.3, 109.2)
- moved C3 8.13 mm to (163.2, 108.0)
- moved C5 8.13 mm to (160.7, 120.0)
- moved C6 8.13 mm to (160.7, 117.5)
- moved D1 8.13 mm to (154.3, 124.5)
- moved D2 8.13 mm to (149.2, 124.5)
- moved D3 8.13 mm to (166.4, 95.9)
- moved FB1 8.13 mm to (170.8, 101.0)
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